File: board/door.sch (EAGLE design)
At the start: 15 parts, among them IC1 7805T

Commit message: add user_button
Parts:
- removed IC1: 7805T, linear4:7805T
- added IC3: 7805, VoltageRegulator:7805
- added S3: (no value), switch-omron:10-XX
Connections:
- new net IO14: JP1.3, S3.S, S3.S1
- net +3V3: now also IC3.OUT; no longer IC1.VO
- net +8V: now also IC3.IN; no longer IC1.VI
- net GND: now also IC3.GND, S3.P, S3.P1; no longer IC1.GND
Changed lines of the file:
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@@
 <setting verticaltext="up"/>
 </settings>
-<grid distance="0.1" unitdist="inch" unit="inch" style="lines" multiple="1" display="no" altdistance="0.01" altunitdist="inch" altunit="inch"/>
+<grid distance="0.05" unitdist="inch" unit="inch" style="lines" multiple="1" display="no" altdistance="0.01" altunitdist="inch" altunit="inch"/>
 <layers>
 <layer number="1" name="Top" color="4" fill="1" visible="no" active="no"/>
@@
 <layer number="111" name="LPC17xx" color="7" fill="1" visible="yes" active="yes"/>
 <layer number="112" name="tSilk" color="7" fill="1" visible="yes" active="yes"/>
+<layer number="113" name="IDFDebug" color="7" fill="1" visible="yes" active="yes"/>
 <layer number="116" name="Patch_BOT" color="9" fill="4" visible="yes" active="yes"/>
 <layer number="118" name="Rect_Pads" color="7" fill="1" visible="no" active="no"/>
@@
 <part name="SUPPLY1" library="supply2" deviceset="+8V" device=""/>
 <part name="+3V4" library="supply1" deviceset="+3V3" device=""/>
-<part name="IC1" library="linear4" deviceset="78*" device="T" technology="05"/>
 <part name="GND8" library="supply1" deviceset="GND" device=""/>
 <part name="C3" library="rcl" deviceset="C-EU" device="050-024X044"/>
@@
 <part name="C7" library="rcl" deviceset="CPOL-EU" device="E5-4"/>
 <part name="GND10" library="supply1" deviceset="GND" device=""/>
+<part name="S3" library="switch-omron" deviceset="10-XX" device=""/>
+<part name="GND14" library="supply1" deviceset="GND" device=""/>
+<part name="IC3" library="VoltageRegulator" deviceset="78*" device="" technology="05"/>
 </parts>
 <sheets>
@@
 <instance part="SUPPLY1" gate="+8V" x="-5.08" y="53.34"/>
 <instance part="+3V4" gate="G$1" x="81.28" y="33.02"/>
-<instance part="IC1" gate="A1" x="58.42" y="30.48"/>
 <instance part="GND8" gate="1" x="58.42" y="7.62"/>
 <instance part="C3" gate="G$1" x="45.72" y="22.86"/>
@@
 <instance part="C7" gate="G$1" x="76.2" y="22.86"/>
 <instance part="GND10" gate="1" x="12.7" y="10.16"/>
+<instance part="S3" gate="1" x="124.46" y="20.32"/>
+<instance part="GND14" gate="1" x="124.46" y="7.62"/>
+<instance part="IC3" gate="G$1" x="58.42" y="30.48"/>
 </instances>
 <busses>
@@
 </segment>
 <segment>
-<pinref part="IC1" gate="A1" pin="VI"/>
 <wire x1="35.56" y1="30.48" x2="38.1" y2="30.48" width="0.1524" layer="91"/>
 <pinref part="C3" gate="G$1" pin="1"/>
 <wire x1="38.1" y1="30.48" x2="45.72" y2="30.48" width="0.1524" layer="91"/>
-<wire x1="45.72" y1="30.48" x2="48.26" y2="30.48" width="0.1524" layer="91"/>
 <wire x1="45.72" y1="30.48" x2="45.72" y2="25.4" width="0.1524" layer="91"/>
 <wire x1="38.1" y1="25.4" x2="38.1" y2="30.48" width="0.1524" layer="91"/>
 <pinref part="SUPPLY2" gate="+8V" pin="+8V"/>
 <pinref part="C6" gate="G$1" pin="+"/>
+<pinref part="IC3" gate="G$1" pin="IN"/>
+<wire x1="45.72" y1="30.48" x2="50.8" y2="30.48" width="0.1524" layer="91"/>
 </segment>
 </net>
@@
 </segment>
 <segment>
-<pinref part="IC1" gate="A1" pin="GND"/>
 <pinref part="GND8" gate="1" pin="GND"/>
 <wire x1="58.42" y1="10.16" x2="58.42" y2="12.7" width="0.1524" layer="91"/>
@@
 <pinref part="C6" gate="G$1" pin="-"/>
 <pinref part="C7" gate="G$1" pin="-"/>
+<pinref part="IC3" gate="G$1" pin="GND"/>
 </segment>
 <segment>
@@
 <wire x1="12.7" y1="12.7" x2="20.32" y2="12.7" width="0.1524" layer="91"/>
 </segment>
+<segment>
+<pinref part="S3" gate="1" pin="P"/>
+<wire x1="124.46" y1="15.24" x2="124.46" y2="10.16" width="0.1524" layer="91"/>
+<pinref part="GND14" gate="1" pin="GND"/>
+<pinref part="S3" gate="1" pin="P1"/>
+<wire x1="124.46" y1="15.24" x2="127" y2="15.24" width="0.1524" layer="91"/>
+</segment>
 </net>
 <net name="+3V3" class="0">
 <segment>
-<pinref part="IC1" gate="A1" pin="VO"/>
 <pinref part="+3V4" gate="G$1" pin="+3V3"/>
 <wire x1="81.28" y1="30.48" x2="76.2" y2="30.48" width="0.1524" layer="91"/>
@@
 <wire x1="76.2" y1="25.4" x2="76.2" y2="30.48" width="0.1524" layer="91"/>
 <pinref part="C7" gate="G$1" pin="+"/>
+<pinref part="IC3" gate="G$1" pin="OUT"/>
+<wire x1="66.04" y1="30.48" x2="68.58" y2="30.48" width="0.1524" layer="91"/>
 </segment>
 <segment>
@@
 </segment>
 </net>
+<net name="IO14" class="0">
+<segment>
+<pinref part="JP1" gate="A" pin="3"/>
+<wire x1="2.54" y1="27.94" x2="-7.62" y2="27.94" width="0.1524" layer="91"/>
+<label x="-7.62" y="27.94" size="1.778" layer="95"/>
+</segment>
+<segment>
+<pinref part="S3" gate="1" pin="S"/>
+<wire x1="124.46" y1="25.4" x2="124.46" y2="38.1" width="0.1524" layer="91"/>
+<label x="124.46" y="33.02" size="1.778" layer="95" rot="R90"/>
+<pinref part="S3" gate="1" pin="S1"/>
+<wire x1="124.46" y1="25.4" x2="127" y2="25.4" width="0.1524" layer="91"/>
+</segment>
+</net>
